Commit message: joystic

File: description/robot_core.xacro (robot description, xacro)
@@ -16,4 +16,12 @@
 <!-- BASE LINK-->
     <link name="base_link">
+    </link>
+<!-- base footprint -->
+    <joint name="base_footprint_joint" type="fixed">
+        <parent link="base_link"/>
+        <child link="base_footprint"/>
+        <origin xyz="0 0 0" rpy="0 0 0"/>
+    </joint>
+    <link name="base_footprint">
     </link>
 <!-- CHASSIS LINK-->
@@ -37,11 +45,9 @@
             </geometry>
         </collision>
-        <xacro:inertial_box mass="0.5" x="0.22" y="0.12" z="0.04">
+        <!-- <xacro:inertial_box mass="0.5" x="0.22" y="0.12" z="0.04">
             <origin xyz="0.11 0 0" rpy="0 0 0 "/>
-        </xacro:inertial_box>
+        </xacro:inertial_box> -->
     </link>
     <gazebo reference="chassis">
-        <mu1>0.2</mu1>
-        <mu2>0.2</mu2>
         <material>Gazebo/White</material>
     </gazebo>
@@ -62,10 +68,10 @@
         <collision>
             <geometry>
-                <sphere  radius="0.032"/>
+                <cylinder  radius="0.032" length="0.03"/>
             </geometry>
         </collision>
-        <xacro:inertial_cylinder mass="0.1" length="0.03" radius="0.032">
+        <!-- <xacro:inertial_cylinder mass="0.1" length="0.03" radius="0.032">
             <origin xyz="0 0. 0" rpy="0 0 0"/>
-        </xacro:inertial_cylinder>
+        </xacro:inertial_cylinder>   -->
     </link>
     <gazebo reference="left_back_wheel">
@@ -88,10 +94,10 @@
         <collision>
             <geometry>
-                <sphere  radius="0.032"/>
+                <cylinder  radius="0.032 " length="0.03"/>
             </geometry>
         </collision>
-        <xacro:inertial_cylinder mass="0.1" length="0.03" radius="0.032">
+        <!-- <xacro:inertial_cylinder mass="0.1" length="0.03" radius="0.032">
             <origin xyz="0 0. 0" rpy="0 0 0"/>
-        </xacro:inertial_cylinder>
+        </xacro:inertial_cylinder>  -->
     </link>
     <gazebo reference="right_back_wheel">
@@ -122,6 +128,6 @@
     </link>
     <gazebo reference="cast_wheel">
-        <mu1>0.2</mu1>
-        <mu2>0.2</mu2>
+        <!-- <mu1>0.2</mu1>
+        <mu2>0.2</mu2> -->
         <material>Gazebo/Black</material>
     </gazebo>

File: description/ros2_control.xacro (robot description, xacro)
@@ -10,5 +10,5 @@
         <param name="baud_rate">57600</param>
         <param name="timeout_ms">1000</param>
-        <param name="enc_counts_per_rev">1240</param>
+        <param name="enc_counts_per_rev">24</param>
     </hardware>
     <joint name="left_back_wheel_joint">
@@ -29,6 +29,5 @@
     </joint>
 </ros2_control>
-<!--
-<ros2_control name="GazeboSystem" type="system">
+<!-- <ros2_control name="GazeboSystem" type="system">
     <hardware>
         <plugin>gazebo_ros2_control/GazeboSystem</plugin>
@@ -50,5 +49,5 @@
         <state_interface name="position"/>
     </joint>
-</ros2_control> -->
+</ros2_control>  -->
 <gazebo>
     <plugin name="gazebo_ros2_control" filename="libgazebo_ros2_control.so">
